File: cpu.sch (KiCad schematic (older format))
At the start: 35 parts, among them P542 TP4, P543 TP5, P545 TP7, P546 TP8, P547 TP9, P548 TP10, P592 UART1, P593 SWD, SW503 DFU, SW514 RESET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

Commit message: [enhancement] Rework cw308 trigger con.
Parts:
- removed JP100: BOOT1, Connector_PinHeader_2.54mm:PinHeader_1x02_P2.54mm_Vertical, symbol Device:Jumper_NO_Small
- removed JP101: BOOT0, Connector_PinHeader_2.54mm:PinHeader_1x02_P2.54mm_Vertical, symbol Device:Jumper_NO_Small
- removed R104: 470, Resistor_SMD:R_0603_1608Metric, symbol Device:R_Small
Connections:
- net BOOT0 is gone; now on net DFU: U500.94 (BOOT0)
- net BOOT1: now also R100.2
- net DFU: no longer U500.30 (PA5)
- net CW_TRIG: now reaches U500.41 (PE10)
- no-connect marks 55 -> 54
Other:
- moved on the sheet: R503, SW503
Changed lines of the file:
@@
 Comment4 ""
 $EndDescr
-$Comp
-L Device:R_Small R104
-U 1 1 557FEF49
-P 1450 5650
-F 0 "R104" V 1530 5650 50  0000 C CNN
-F 1 "470" V 1450 5650 50  0000 C CNN
-F 2 "Resistor_SMD:R_0603_1608Metric" V 1380 5650 30  0001 C CNN
-F 3 "" H 1450 5650 30  0000 C CNN
-F 4 "Farnell" H 0   0   50  0001 C CNN "Distrib"
-F 5 "Farnell" H 0   0   50  0001 C CNN "Distrib Name"
-F 6 "1469815" H 0   0   50  0001 C CNN "Distrib PN"
-F 7 "1469815" H 0   0   50  0001 C CNN "Distrib Part Num"
-F 8 "Vishay" H 0   0   50  0001 C CNN "MFG Name"
-F 9 "CRCW0603470RFKEA" H 0   0   50  0001 C CNN "MFG Part Num"
-	1    1450 5650
-	1    0    0    -1
-$EndComp
-Text Label 1550 4950 0    60   ~ 0
-BOOT0
 Text Label 1550 4750 0    60   ~ 0
 BOOT1
@@
 	1    0    0    -1
 $EndComp
-Text Label 8850 5750 0    60   ~ 0
-BOOT0
 Text Label 8850 9300 0    60   ~ 0
 BOOT1
@@
 NoConn ~ 12600 6300
 NoConn ~ 12600 6400
-NoConn ~ 12600 6500
 NoConn ~ 9650 6500
 $Comp
@@
 L Switch:SW_Push SW503
 U 1 1 58BDB2DF
-P 5200 4500
-F 0 "SW503" H 5350 4610 50  0000 C CNN
-F 1 "DFU" H 5200 4420 50  0000 C CNN
-F 2 "leia:KSR_TACTILE_SWITCH" H 5200 4500 60  0001 C CNN
-F 3 "http://www.farnell.com/datasheets/1780692.pdf" H 5200 4500 60  0001 C CNN
-F 4 "C & K COMPONENTS" H 5200 4500 60  0001 C CNN "MFG Name"
-F 5 "KSR231G LFS" H 5200 4500 60  0001 C CNN "MFG Part Num"
-F 6 "1201422" H 5200 4500 60  0001 C CNN "Distrib PN"
-F 7 "Farnell" H 5200 4500 50  0001 C CNN "Distrib"
-F 8 "http://fr.farnell.com/c-k-components/ksr231g-lfs/tactile-commutateur-miniature/dp/1201422" H 5200 4500 60  0001 C CNN "Distrib Link"
-F 9 "Farnell" H 0   0   50  0001 C CNN "Distrib Name"
-	1    5200 4500
+P 1200 5000
+F 0 "SW503" H 1350 5110 50  0000 C CNN
+F 1 "DFU" H 1200 4920 50  0000 C CNN
+F 2 "leia:KSR_TACTILE_SWITCH" H 1200 5000 60  0001 C CNN
+F 3 "http://www.farnell.com/datasheets/1780692.pdf" H 1200 5000 60  0001 C CNN
+F 4 "C & K COMPONENTS" H 1200 5000 60  0001 C CNN "MFG Name"
+F 5 "KSR231G LFS" H 1200 5000 60  0001 C CNN "MFG Part Num"
+F 6 "1201422" H 1200 5000 60  0001 C CNN "Distrib PN"
+F 7 "Farnell" H 1200 5000 50  0001 C CNN "Distrib"
+F 8 "http://fr.farnell.com/c-k-components/ksr231g-lfs/tactile-commutateur-miniature/dp/1201422" H 1200 5000 60  0001 C CNN "Distrib Link"
+F 9 "Farnell" H -4000 500 50  0001 C CNN "Distrib Name"
+	1    1200 5000
 	0    -1   1    0
 $EndComp
@@
 L Device:R_Small R503
 U 1 1 58BDBDAB
-P 5200 5050
-F 0 "R503" V 5280 5050 50  0000 C CNN
-F 1 "10K" V 5200 5050 50  0000 C CNN
-F 2 "Resistor_SMD:R_0603_1608Metric" V 5130 5050 30  0001 C CNN
-F 3 "" H 5200 5050 30  0000 C CNN
-F 4 "Farnell" H 0   0   50  0001 C CNN "Distrib"
-F 5 "Farnell" H 0   0   50  0001 C CNN "Distrib Name"
-F 6 "1738918" H 0   0   50  0001 C CNN "Distrib PN"
-F 7 "1738918" H 0   0   50  0001 C CNN "Distrib Part Num"
-F 8 "Vishay" H 0   0   50  0001 C CNN "MFG Name"
-F 9 "CRCW060310K0FKEAHP" H 0   0   50  0001 C CNN "MFG Part Num"
-	1    5200 5050
-	1    0    0    -1
-$EndComp
-Text Label 5700 4850 0    60   ~ 0
+P 1200 5550
+F 0 "R503" V 1280 5550 50  0000 C CNN
+F 1 "10K" V 1200 5550 50  0000 C CNN
+F 2 "Resistor_SMD:R_0603_1608Metric" V 1130 5550 30  0001 C CNN
+F 3 "" H 1200 5550 30  0000 C CNN
+F 4 "Farnell" H -4000 500 50  0001 C CNN "Distrib"
+F 5 "Farnell" H -4000 500 50  0001 C CNN "Distrib Name"
+F 6 "1738918" H -4000 500 50  0001 C CNN "Distrib PN"
+F 7 "1738918" H -4000 500 50  0001 C CNN "Distrib Part Num"
+F 8 "Vishay" H -4000 500 50  0001 C CNN "MFG Name"
+F 9 "CRCW060310K0FKEAHP" H -4000 500 50  0001 C CNN "MFG Part Num"
+	1    1200 5550
+	1    0    0    -1
+$EndComp
+Text Label 1700 5350 0    60   ~ 0
 DFU
-Text Label 9050 7800 2    60   ~ 0
+Text Label 8950 5750 2    60   ~ 0
 DFU
 Text Notes 900  6450 0    60   ~ 0
@@
 	12600 6600 13550 6600
 Wire Wire Line
-	1450 4950 2050 4950
-Wire Wire Line
 	3150 4250 4200 4250
 Wire Wire Line
@@
 Wire Wire Line
 	8350 5900 9650 5900
-Wire Wire Line
-	9650 5750 8850 5750
 Connection ~ 7950 5700
 Connection ~ 7950 5100
@@
 	20250 4250 19500 4250
 Wire Wire Line
-	5200 4850 5700 4850
-Connection ~ 5200 4850
+	1200 5350 1700 5350
+Connection ~ 1200 5350
 Wire Wire Line
 	12600 8000 14300 8000
@@
 NoConn ~ 9650 8300
 NoConn ~ 12600 8800
-$Comp
-L Device:Jumper_NO_Small JP101
-U 1 1 5C4FF62B
-P 1450 5350
-F 0 "JP101" V 1404 5398 50  0000 L CNN
-F 1 "BOOT0" V 1495 5398 50  0000 L CNN
-F 2 "Connector_PinHeader_2.54mm:PinHeader_1x02_P2.54mm_Vertical" H 1450 5350 50  0001 C CNN
-F 3 "~" H 1450 5350 50  0001 C CNN
-F 4 "Molex" V 1450 5350 50  0001 C CNN "MFG Name"
-F 5 "90120-0762" V 1450 5350 50  0001 C CNN "MFG Part Num"
-F 6 "2751456" V 1450 5350 50  0001 C CNN "Distrib PN"
-F 7 "Farnell" V 1450 5350 50  0001 C CNN "Distrib"
-F 8 "Farnell" H 0   0   50  0001 C CNN "Distrib Name"
-	1    1450 5350
-	0    1    1    0
-$EndComp
-$Comp
-L Device:Jumper_NO_Small JP100
-U 1 1 5C5084C4
-P 1450 4600
-F 0 "JP100" V 1404 4648 50  0000 L CNN
-F 1 "BOOT1" V 1495 4648 50  0000 L CNN
-F 2 "Connector_PinHeader_2.54mm:PinHeader_1x02_P2.54mm_Vertical" H 1450 4600 50  0001 C CNN
-F 3 "~" H 1450 4600 50  0001 C CNN
-F 4 "Molex" V 1450 4600 50  0001 C CNN "MFG Name"
-F 5 "90120-0762" V 1450 4600 50  0001 C CNN "MFG Part Num"
-F 6 "2751456" V 1450 4600 50  0001 C CNN "Distrib PN"
-F 7 "Farnell" V 1450 4600 50  0001 C CNN "Distrib"
-F 8 "Farnell" H 0   0   50  0001 C CNN "Distrib Name"
-	1    1450 4600
-	0    1    1    0
-$EndComp
-Wire Wire Line
-	1450 4750 1450 4700
-Wire Wire Line
-	1450 4950 1450 5250
-Wire Wire Line
-	9650 7800 9050 7800
+Wire Wire Line
+	9650 5750 8950 5750
 NoConn ~ 12600 8700
 Wire Wire Line
@@
 Wire Wire Line
 	5000 2600 5000 2450
-$Comp
-L power:GNDD #PWR0128
-U 1 1 5C5A9F08
-P 1450 5900
-F 0 "#PWR0128" H 1450 5650 50  0001 C CNN
-F 1 "GNDD" H 1454 5745 50  0000 C CNN
-F 2 "" H 1450 5900 50  0001 C CNN
-F 3 "" H 1450 5900 50  0001 C CNN
-	1    1450 5900
-	1    0    0    -1
-$EndComp
 $Comp
 L power:GNDD #PWR0129
@@
 L power:GNDD #PWR0131
 U 1 1 5C5BB295
-P 5200 5300
-F 0 "#PWR0131" H 5200 5050 50  0001 C CNN
-F 1 "GNDD" H 5204 5145 50  0000 C CNN
-F 2 "" H 5200 5300 50  0001 C CNN
-F 3 "" H 5200 5300 50  0001 C CNN
-	1    5200 5300
+P 1200 5800
+F 0 "#PWR0131" H 1200 5550 50  0001 C CNN
+F 1 "GNDD" H 1204 5645 50  0000 C CNN
+F 2 "" H 1200 5800 50  0001 C CNN
+F 3 "" H 1200 5800 50  0001 C CNN
+	1    1200 5800
 	1    0    0    -1
 $EndComp
@@
 L power:VDD #PWR0140
 U 1 1 5C6A853C
-P 5200 4100
-F 0 "#PWR0140" H 5200 3950 50  0001 C CNN
-F 1 "VDD" H 5217 4273 50  0000 C CNN
-F 2 "" H 5200 4100 50  0001 C CNN
-F 3 "" H 5200 4100 50  0001 C CNN
-	1    5200 4100
+P 1200 4600
+F 0 "#PWR0140" H 1200 4450 50  0001 C CNN
+F 1 "VDD" H 1217 4773 50  0000 C CNN
+F 2 "" H 1200 4600 50  0001 C CNN
+F 3 "" H 1200 4600 50  0001 C CNN
+	1    1200 4600
 	1    0    0    -1
 $EndComp
@@
 Wire Wire Line
 	7900 7500 9650 7500
-NoConn ~ 9650 7600
 NoConn ~ 9650 7900
 NoConn ~ 9650 8000
@@
 	1450 4200 1450 4150
 Wire Wire Line
-	1450 4400 1450 4500
-Wire Wire Line
-	1450 5450 1450 5550
-Wire Wire Line
-	1450 5750 1450 5900
-Wire Wire Line
 	2900 5050 2900 5300
 Wire Wire Line
@@
 	3500 4450 3500 4850
 Wire Wire Line
-	5200 4850 5200 4950
-Wire Wire Line
-	5200 5150 5200 5300
+	1200 5350 1200 5450
+Wire Wire Line
+	1200 5650 1200 5800
 Wire Wire Line
 	7950 5000 7950 5100
@@
 	7650 5600 7650 5700
 Wire Wire Line
-	5200 4100 5200 4300
-Wire Wire Line
-	5200 4700 5200 4850
+	1200 4600 1200 4800
+Wire Wire Line
+	1200 5200 1200 5350
 Wire Wire Line
 	9650 9500 8850 9500
 Text Label 8850 9500 0    60   ~ 0
 UART2_CARD_CLK
+Text HLabel 14400 6500 2    50   Output ~ 0
+CW_TRIG
+Wire Wire Line
+	12600 6500 14400 6500
+NoConn ~ 9650 7600
+Wire Wire Line
+	1450 4400 1450 4750
 $EndSCHEMATC

Commit message: [enhancement] add HSE
Parts:
- added C4005: 0.01uF, Capacitor_SMD:C_0603_1608Metric, symbol Device:C_Small
- added P4001: XI, TestPoint:TestPoint_Pad_D1.0mm, symbol Connector_Generic:Conn_01x01
- added Y4001: ASEMB-16.000MHZ-LY-T, Oscillator:Oscillator_SMD_Abracon_ASE-4Pin_3.2x2.5mm, symbol leia:ASE-xxxMHz-Oscillator
Connections:
- net CARD_CLK: now also U500.26 (PA3); no longer U500.90 (PB4)
- net GNDD: now also C4005.2, Y4001.2 (GND)
- net VDD: now also C4005.1, Y4001.1 (STBY), Y4001.4 (Vdd)
- net at U500.12 (PH0): now also P4001.1 (Pin_1), Y4001.3 (OUT)
- no-connect marks 54 -> 53
Other:
- note added: "PA4 is used when the smartcard is driven with the hardware block\nPA3 is used in BitBang mode"
- note added: "see qtzcry-app-notes.pdf (in datasheets)"
- moved on the sheet: C500, C506, C511, C514, C519, C521, C522, C528, C549, C550, C573, C575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

Commit message: [Fix] General cleanup before production
Connections:
- net BOOT1: now also R100.1; no longer R100.2
- net GNDD: now also R100.2
- net VDD: no longer R100.1
Other:
- moved on the sheet: R100
Changed lines of the file:
@@
 Comment4 ""
 $EndDescr
-Text Label 2450 4650 0    60   ~ 0
+Text Label 2750 5300 0    60   ~ 0
 BOOT1
 $Comp
@@
 	1    0    0    -1
 $EndComp
-Text Label 2600 5250 0    60   ~ 0
+Text Label 2750 5100 0    60   ~ 0
 DFU
 Text Label 9850 5650 2    60   ~ 0
@@
 	4400 4350 5100 4350
 Wire Wire Line
-	2350 4650 2950 4650
+	2350 5300 2750 5300
 Wire Notes Line
 	22000 6800 22000 2000
@@
 	21150 4150 20400 4150
 Wire Wire Line
-	2100 5250 2600 5250
-Connection ~ 2100 5250
+	2100 5100 2750 5100
+Connection ~ 2100 5100
 Wire Wire Line
 	13500 7900 15200 7900
@@
 $EndComp
 $Comp
-L power:VDD #PWR0139
-U 1 1 5C6A7F4D
-P 2350 4050
-F 0 "#PWR0139" H 2350 3900 50  0001 C CNN
-F 1 "VDD" H 2367 4223 50  0000 C CNN
-F 2 "" H 2350 4050 50  0001 C CNN
-F 3 "" H 2350 4050 50  0001 C CNN
-	1    2350 4050
-	1    0    0    -1
-$EndComp
-$Comp
 L power:VDD #PWR0140
 U 1 1 5C6A853C
@@
 L Device:R_Small R100
 U 1 1 557FEE42
-P 2350 4200
-F 0 "R100" V 2430 4200 50  0000 C CNN
-F 1 "10K" V 2350 4200 50  0000 C CNN
-F 2 "Resistor_SMD:R_0603_1608Metric" V 2280 4200 30  0001 C CNN
-F 3 "" H 2350 4200 30  0000 C CNN
-F 4 "Farnell" H 900 -100 50  0001 C CNN "Distrib"
-F 5 "Farnell" H 900 -100 50  0001 C CNN "Distrib Name"
-F 6 "1738918" H 900 -100 50  0001 C CNN "Distrib PN"
-F 7 "1738918" H 900 -100 50  0001 C CNN "Distrib Part Num"
-F 8 "Vishay" H 900 -100 50  0001 C CNN "MFG Name"
-F 9 "CRCW060310K0FKEAHP" H 900 -100 50  0001 C CNN "MFG Part Num"
-	1    2350 4200
+P 2350 5450
+F 0 "R100" V 2430 5450 50  0000 C CNN
+F 1 "10K" V 2350 5450 50  0000 C CNN
+F 2 "Resistor_SMD:R_0603_1608Metric" V 2280 5450 30  0001 C CNN
+F 3 "" H 2350 5450 30  0000 C CNN
+F 4 "Farnell" H 900 1150 50  0001 C CNN "Distrib"
+F 5 "Farnell" H 900 1150 50  0001 C CNN "Distrib Name"
+F 6 "1738918" H 900 1150 50  0001 C CNN "Distrib PN"
+F 7 "1738918" H 900 1150 50  0001 C CNN "Distrib Part Num"
+F 8 "Vishay" H 900 1150 50  0001 C CNN "MFG Name"
+F 9 "CRCW060310K0FKEAHP" H 900 1150 50  0001 C CNN "MFG Part Num"
+	1    2350 5450
 	1    0    0    -1
 $EndComp
@@
 	7900 5000 8550 5000
 Wire Wire Line
-	2350 4100 2350 4050
+	2350 5350 2350 5300
 Wire Wire Line
 	3800 4950 3800 5200
@@
 	4400 4350 4400 4750
 Wire Wire Line
-	2100 5250 2100 5350
-Wire Wire Line
-	2100 5550 2100 5700
+	2100 5100 2100 5350
+Wire Wire Line
+	2100 5550 2100 5650
 Wire Wire Line
 	8850 4900 8850 5000
@@
 Wire Wire Line
 	2100 4500 2100 4700
-Wire Wire Line
-	2100 5100 2100 5250
 Text HLabel 15300 6400 2    50   Output ~ 0
 CW_TRIG
 Wire Wire Line
 	13500 6400 15300 6400
-Wire Wire Line
-	2350 4300 2350 4650
 Wire Wire Line
 	10550 7500 9650 7500
@@
 	1    0    0    -1
 $EndComp
+Wire Wire Line
+	2100 5650 2350 5650
+Wire Wire Line
+	2350 5650 2350 5550
+Connection ~ 2100 5650
+Wire Wire Line
+	2100 5650 2100 5700
 $EndSCHEMATC
