File: leia.sch (KiCad schematic (older format))
At the start: 27 parts, among them J1002 READER_GND, J1003 READER_VDD, J1101 TARGET_PWR, J1102 TARGET_GND, J1103 TARGET_EXT_PWR, J1112 TARGET_SHUNT, J6 EXT_READER_VCC, P523 CMD, U520 FOD8012A

Commit message: [enhancement] Add tests points for smartcard controlled triggers, connect PB4 to CARD_CLK for bitbanging mode
Parts:
- added D1001: VDDA, LED_SMD:LED_0603_1608Metric_Castellated, symbol Device:LED_ALT
- added R1002: 470, Resistor_SMD:R_0603_1608Metric, symbol Device:R_Small
Connections:
- net labels added: GND_UART, VDD_UART
- wire segments 138 -> 147
Other:
- moved on the sheet: FID1005
Changed lines of the file:
@@
 NoConn ~ 13700 8800
 NoConn ~ 13350 8800
-Text Label 15400 5050 2    50   ~ 0
+Text Label 15250 5050 2    50   ~ 0
 CW_PWR
 Text Label 15300 7350 2    50   ~ 0
@@
 	6800 4950 7900 4950
 Wire Wire Line
-	14850 5050 15400 5050
-Wire Wire Line
-	14850 5800 15150 5800
+	14850 5050 15250 5050
+Wire Wire Line
+	14850 5550 15150 5550
 Text Label 5150 8750 2    50   ~ 0
 CW_PWR
@@
 L leia:Mechanical_Fiducial FID1005
 U 1 1 5CCA9D97
-P 15150 8650
-F 0 "FID1005" H 15150 8450 60  0000 C CNN
-F 1 "FIDUCIAL-RESCUE-rescue" H 15150 8800 60  0001 C CNN
-F 2 "Fiducial:Fiducial_1mm_Mask2mm" H 15150 8650 60  0001 C CNN
-F 3 "" H 15150 8650 60  0000 C CNN
-	1    15150 8650
+P 15100 8650
+F 0 "FID1005" H 15100 8450 60  0000 C CNN
+F 1 "FIDUCIAL-RESCUE-rescue" H 15100 8800 60  0001 C CNN
+F 2 "Fiducial:Fiducial_1mm_Mask2mm" H 15100 8650 60  0001 C CNN
+F 3 "" H 15100 8650 60  0000 C CNN
+	1    15100 8650
 	1    0    0    -1
 $EndComp
@@
 	12450 3650 12450 2900
 Wire Wire Line
-	13800 3650 14200 3650
+	13800 3650 13950 3650
 Wire Wire Line
 	13800 3950 14100 3950
@@
 Connection ~ 14200 3650
 Wire Wire Line
-	14100 3950 14850 3950
+	14100 3950 14200 3950
 Wire Wire Line
 	14200 3650 14850 3650
@@
 	12750 3750 13000 3750
 Wire Wire Line
-	15350 3950 15750 3950
-Wire Wire Line
-	15350 3650 15750 3650
+	15350 3950 15650 3950
+Wire Wire Line
+	15350 3650 15650 3650
 Wire Wire Line
 	15350 3750 15500 3750
@@
 F4 "TARGET_GND" U R 14850 7350 50
 F5 "TARGET_PWR" U R 14850 5050 50
-F6 "VREF" O R 14850 5800 50
+F6 "VREF" O R 14850 5550 50
+F7 "GNDREF" I R 14850 5700 50
+F8 "VDD_UART" I R 14850 6200 50
+F9 "GND_UART" I R 14850 6300 50
 $EndSheet
 $Sheet
@@
 	6650 7150 6650 8550
 $Comp
-L power:GNDA #PWR?
-U 1 1 5CCB43C6
-P 15750 4000
-AR Path="/5B19B7B2/5CCB43C6" Ref="#PWR?"  Part="1"
-AR Path="/5CD07BF2/5CCB43C6" Ref="#PWR?"  Part="1"
-AR Path="/5CCB43C6" Ref="#PWR0154"  Part="1"
-AR Path="/5CBC3017/5CCB43C6" Ref="#PWR0154"  Part="1"
-F 0 "#PWR0154" H 15750 3750 50  0001 C CNN
-F 1 "GNDA" H 15755 3827 50  0000 C CNN
-F 2 "" H 15750 4000 50  0001 C CNN
-F 3 "" H 15750 4000 50  0001 C CNN
-	1    15750 4000
-	1    0    0    -1
-$EndComp
-Wire Wire Line
-	15750 4000 15750 3950
-$Comp
-L power:VDDA #PWR?
-U 1 1 5CCC7BEB
-P 15750 3550
-AR Path="/5B19B7B2/5CCC7BEB" Ref="#PWR?"  Part="1"
-AR Path="/5CD07BF2/5CCC7BEB" Ref="#PWR?"  Part="1"
-AR Path="/5CCC7BEB" Ref="#PWR0155"  Part="1"
-AR Path="/5CBC3017/5CCC7BEB" Ref="#PWR0155"  Part="1"
-F 0 "#PWR0155" H 15750 3400 50  0001 C CNN
-F 1 "VDDA" H 15750 3750 50  0000 C CNN
-F 2 "" H 15750 3550 50  0001 C CNN
-F 3 "" H 15750 3550 50  0001 C CNN
-F 4 "" H 11300 7450 50  0001 C CNN "MFG Name"
-F 5 "" H 11300 7450 50  0001 C CNN "MFG Part Num"
-F 6 "" H 11300 7450 50  0001 C CNN "Distrib Name"
-F 7 "" H 11300 7450 50  0001 C CNN "Distrib Part Num"
-	1    15750 3550
-	1    0    0    -1
-$EndComp
-Wire Wire Line
-	15750 3550 15750 3650
-$Comp
 L power:VDDA #PWR?
 U 1 1 5CCEDA52
-P 15150 5650
+P 15150 5400
 AR Path="/5B19B7B2/5CCEDA52" Ref="#PWR?"  Part="1"
 AR Path="/5CD07BF2/5CCEDA52" Ref="#PWR?"  Part="1"
 AR Path="/5CCEDA52" Ref="#PWR0156"  Part="1"
 AR Path="/5CBC3017/5CCEDA52" Ref="#PWR0156"  Part="1"
-F 0 "#PWR0156" H 15150 5500 50  0001 C CNN
-F 1 "VDDA" H 15150 5850 50  0000 C CNN
-F 2 "" H 15150 5650 50  0001 C CNN
-F 3 "" H 15150 5650 50  0001 C CNN
-F 4 "" H 10700 9550 50  0001 C CNN "MFG Name"
-F 5 "" H 10700 9550 50  0001 C CNN "MFG Part Num"
-F 6 "" H 10700 9550 50  0001 C CNN "Distrib Name"
-F 7 "" H 10700 9550 50  0001 C CNN "Distrib Part Num"
-	1    15150 5650
-	1    0    0    -1
-$EndComp
-Wire Wire Line
-	15150 5650 15150 5800
+F 0 "#PWR0156" H 15150 5250 50  0001 C CNN
+F 1 "VDDA" H 15150 5600 50  0000 C CNN
+F 2 "" H 15150 5400 50  0001 C CNN
+F 3 "" H 15150 5400 50  0001 C CNN
+F 4 "" H 10700 9300 50  0001 C CNN "MFG Name"
+F 5 "" H 10700 9300 50  0001 C CNN "MFG Part Num"
+F 6 "" H 10700 9300 50  0001 C CNN "Distrib Name"
+F 7 "" H 10700 9300 50  0001 C CNN "Distrib Part Num"
+	1    15150 5400
+	1    0    0    -1
+$EndComp
+Wire Wire Line
+	15150 5400 15150 5550
 Wire Wire Line
 	7700 10250 8150 10250
@@
 Wire Wire Line
 	2200 7800 2200 9000
+$Comp
+L Device:LED_ALT D?
+U 1 1 5CFF716D
+P 13950 4450
+AR Path="/5B22B7CD/5CFF716D" Ref="D?"  Part="1"
+AR Path="/5B19B7B2/5CFF716D" Ref="D?"  Part="1"
+AR Path="/5CBC3017/5B19B7B2/5CFF716D" Ref="D?"  Part="1"
+AR Path="/5CFF716D" Ref="D1001"  Part="1"
+F 0 "D1001" H 13950 4550 50  0000 C CNN
+F 1 "VDDA" H 13950 4350 50  0000 C CNN
+F 2 "LED_SMD:LED_0603_1608Metric_Castellated" H 13950 4450 60  0001 C CNN
+F 3 "" H 13950 4450 60  0000 C CNN
+F 4 "Vishay" H 13950 4450 50  0001 C CNN "MFG Name"
+F 5 "TLMS1100-GS08.." H 13950 4450 50  0001 C CNN "MFG Part Num"
+F 6 "1440338" H 13950 4450 50  0001 C CNN "Distrib PN"
+F 7 "https://fr.farnell.com/vishay/tlms1100-gs08/led-red-1-6mm-x-0-8mm-63mcd-633nm/dp/1440338" H 13950 4450 50  0001 C CNN "Distrib Link"
+F 8 "Farnell" H 13950 4450 50  0001 C CNN "Distrib"
+F 9 "Farnell" H 10450 -1000 50  0001 C CNN "Distrib Name"
+	1    13950 4450
+	0    -1   -1   0
+$EndComp
+$Comp
+L Device:R_Small R?
+U 1 1 5CFF7179
+P 13950 4100
+AR Path="/5B22B7CD/5CFF7179" Ref="R?"  Part="1"
+AR Path="/5B19B7B2/5CFF7179" Ref="R?"  Part="1"
+AR Path="/5CBC3017/5B19B7B2/5CFF7179" Ref="R?"  Part="1"
+AR Path="/5CFF7179" Ref="R1002"  Part="1"
+F 0 "R1002" V 14030 4100 50  0000 C CNN
+F 1 "470" V 13950 4100 50  0000 C CNN
+F 2 "Resistor_SMD:R_0603_1608Metric" V 13880 4100 30  0001 C CNN
+F 3 "" H 13950 4100 30  0000 C CNN
+F 4 "Farnell" H 10450 -850 50  0001 C CNN "Distrib"
+F 5 "Farnell" H 10450 -850 50  0001 C CNN "Distrib Name"
+F 6 "1469815" H 10450 -850 50  0001 C CNN "Distrib PN"
+F 7 "1469815" H 10450 -850 50  0001 C CNN "Distrib Part Num"
+F 8 "Vishay" H 10450 -850 50  0001 C CNN "MFG Name"
+F 9 "CRCW0603470RFKEA" H 10450 -850 50  0001 C CNN "MFG Part Num"
+	1    13950 4100
+	1    0    0    -1
+$EndComp
+Wire Wire Line
+	13950 4200 13950 4300
+Wire Wire Line
+	13950 3650 13950 4000
+Connection ~ 13950 3650
+Wire Wire Line
+	13950 3650 14200 3650
+Wire Wire Line
+	13950 4800 14200 4800
+Wire Wire Line
+	14200 4800 14200 3950
+Wire Wire Line
+	13950 4600 13950 4800
+Connection ~ 14200 3950
+Wire Wire Line
+	14200 3950 14850 3950
+Wire Wire Line
+	14850 5700 15150 5700
+Wire Wire Line
+	15150 5700 15150 5900
+$Comp
+L power:GNDA #PWR?
+U 1 1 5CFA7C05
+P 15150 5900
+AR Path="/5B19B7B2/5CFA7C05" Ref="#PWR?"  Part="1"
+AR Path="/5CD07BF2/5CFA7C05" Ref="#PWR?"  Part="1"
+AR Path="/5CFA7C05" Ref="#PWR0122"  Part="1"
+AR Path="/5CBC3017/5CFA7C05" Ref="#PWR?"  Part="1"
+F 0 "#PWR0122" H 15150 5650 50  0001 C CNN
+F 1 "GNDA" H 15155 5727 50  0000 C CNN
+F 2 "" H 15150 5900 50  0001 C CNN
+F 3 "" H 15150 5900 50  0001 C CNN
+	1    15150 5900
+	1    0    0    -1
+$EndComp
+Text Label 15650 3650 0    50   ~ 0
+VDD_UART
+Text Label 15650 3950 0    50   ~ 0
+GND_UART
+Text Label 15050 6300 0    50   ~ 0
+GND_UART
+Text Label 15050 6200 0    50   ~ 0
+VDD_UART
+Wire Wire Line
+	14850 6200 15050 6200
+Wire Wire Line
+	14850 6300 15050 6300
 $EndSCHEMATC

Commit message: [enhancement] WIP working on power domain isolation
Parts:
- removed J1002: READER_GND, Connector_PinHeader_2.54mm:PinHeader_2x03_P2.54mm_Vertical, symbol Connector_Generic:Conn_02x03_Odd_Even
Connections:
- no-connect marks 7 -> 6
Changed lines of the file:
@@
 	7050 1200 6300 1200
-Wire Wire Line
-	7300 10250 7350 10250
 Wire Wire Line
 	7550 1400 7900 1400
@@
 Wire Wire Line
 	7900 1400 7900 1300
-$Comp
-L Connector_Generic:Conn_02x03_Odd_Even J1002
-U 1 1 5C3ABCFD
-P 7100 10250
-F 0 "J1002" H 7150 10567 50  0000 C CNN
-F 1 "READER_GND" H 7150 10476 50  0000 C CNN
-F 2 "Connector_PinHeader_2.54mm:PinHeader_2x03_P2.54mm_Vertical" H 7100 10250 50  0001 C CNN
-F 3 "~" H 7100 10250 50  0001 C CNN
-F 4 "Molex" H 6650 8200 50  0001 C CNN "MFG Name"
-F 5 "90131-0763" H 6650 8200 50  0001 C CNN "MFG Part Num"
-F 6 "Farnell" H 6650 8200 50  0001 C CNN "Distrib Name"
-F 7 "Farnell" H 850 1050 50  0001 C CNN "Distrib"
-F 8 "9733574" H 850 1050 50  0001 C CNN "Distrib PN"
-	1    7100 10250
-	-1   0    0    -1
-$EndComp
-Wire Wire Line
-	7300 10350 7350 10350
-Text Label 6050 10350 0    50   ~ 0
+Text Label 6050 10250 0    50   ~ 0
 EXT_READER_GND
 Wire Wire Line
@@
 Text Label 6400 1200 0    50   ~ 0
 USB_READER_VCC
-Text Label 6050 10150 0    50   ~ 0
-USB_READER_GND
 $Comp
 L Connector:Conn_Coaxial J6
@@
 Wire Wire Line
 	14850 7350 15300 7350
-Wire Wire Line
-	7350 10350 7350 10250
 Connection ~ 7350 10250
 Text Label 6800 4250 2    50   ~ 0
@@
 Wire Wire Line
 	6050 6800 8150 6800
-Wire Wire Line
-	6050 10350 6800 10350
-Wire Wire Line
-	6050 10150 6800 10150
 $Comp
 L Connector:TestPoint_Alt TP1001
@@
 	12750 3750 13000 3750
 Wire Wire Line
-	15350 3950 15650 3950
-Wire Wire Line
-	15350 3650 15650 3650
+	15350 3950 15400 3950
+Wire Wire Line
+	15350 3650 15400 3650
 Wire Wire Line
 	15350 3750 15500 3750
@@
 VDDD and GNDD are connected to \noptocouplers reader side
 Text Notes 3800 8050 0    50   ~ 0
-User can choose between external \npower supply or CW power supply.
-Text Notes 6050 10650 0    50   ~ 0
 User can choose between external \npower supply or CW power supply.
 Text Notes 6350 800  0    50   ~ 0
@@
 	6300 7450 6300 7350
 Wire Wire Line
-	7300 10150 7350 10150
-Wire Wire Line
-	7350 10150 7350 10250
-NoConn ~ 6800 10250
-Wire Wire Line
 	6300 1200 6300 1550
 Wire Wire Line
@@
 Wire Wire Line
 	14850 6300 15050 6300
+Wire Wire Line
+	7350 10100 6050 10100
+Text Label 6050 10100 0    50   ~ 0
+USB_READER_GND
+Wire Wire Line
+	7350 10100 7350 10250
+Wire Wire Line
+	6050 10250 7350 10250
+$Comp
+L power:GNDA #PWR?
+U 1 1 5D0CC0F2
+P 15400 4450
+AR Path="/5B19B7B2/5D0CC0F2" Ref="#PWR?"  Part="1"
+AR Path="/5CD07BF2/5D0CC0F2" Ref="#PWR?"  Part="1"
+AR Path="/5D0CC0F2" Ref="#PWR0154"  Part="1"
+AR Path="/5CBC3017/5D0CC0F2" Ref="#PWR?"  Part="1"
+F 0 "#PWR0154" H 15400 4200 50  0001 C CNN
+F 1 "GNDA" H 15405 4277 50  0000 C CNN
+F 2 "" H 15400 4450 50  0001 C CNN
+F 3 "" H 15400 4450 50  0001 C CNN
+	1    15400 4450
+	1    0    0    -1
+$EndComp
+Wire Wire Line
+	15400 4450 15400 3950
+Connection ~ 15400 3950
+Wire Wire Line
+	15400 3950 15650 3950
+$Comp
+L power:VDDA #PWR?
+U 1 1 5D0D488A
+P 15400 3400
+AR Path="/5B19B7B2/5D0D488A" Ref="#PWR?"  Part="1"
+AR Path="/5CD07BF2/5D0D488A" Ref="#PWR?"  Part="1"
+AR Path="/5D0D488A" Ref="#PWR?"  Part="1"
+AR Path="/5CBC3017/5D0D488A" Ref="#PWR?"  Part="1"
+F 0 "#PWR?" H 15400 3250 50  0001 C CNN
+F 1 "VDDA" H 15400 3600 50  0000 C CNN
+F 2 "" H 15400 3400 50  0001 C CNN
+F 3 "" H 15400 3400 50  0001 C CNN
+F 4 "" H 10950 7300 50  0001 C CNN "MFG Name"
+F 5 "" H 10950 7300 50  0001 C CNN "MFG Part Num"
+F 6 "" H 10950 7300 50  0001 C CNN "Distrib Name"
+F 7 "" H 10950 7300 50  0001 C CNN "Distrib Part Num"
+	1    15400 3400
+	1    0    0    -1
+$EndComp
+Wire Wire Line
+	15400 3400 15400 3650
+Connection ~ 15400 3650
+Wire Wire Line
+	15400 3650 15650 3650
 $EndSCHEMATC

Commit message: [enhancement] Rework cw308 trigger con.
Parts:
- added C1004, C1005: 0.1uF 35V Tant, Capacitor_Tantalum_SMD:CP_EIA-3216-18_Kemet-A, symbol Device:CP_Small
- added P1001: CMD, Connector_PinHeader_2.54mm:PinHeader_2x02_P2.54mm_Vertical, symbol Connector_Generic:Conn_02x02_Odd_Even
- added U1001: FOD8001, Package_SO:SOIC-8_3.9x4.9mm_P1.27mm, symbol optos:FOD8001
- P523: footprint Connector_PinHeader_2.54mm:PinHeader_2x04_P2.54mm_Vertical -> Connector_PinHeader_2.54mm:PinHeader_2x02_P2.54mm_Vertical; symbol Connector_Generic:Conn_02x04_Odd_Even -> Connector_Generic:Conn_02x02_Odd_Even; Distrib PN 2528034 -> (none); MFG Part Num 826632-4 -> (none)
Connections:
- net labels added: GND_CMD, VDD_CMD
- net labels removed: GND_CONSOLE, GND_UART, VDD_CONSOLE, VDD_UART
- wire segments 147 -> 157
Other:
- moved on the sheet: FID1001, FID1002, FID1003, FID1004, FID1005, FID1006, HOLE1, HOLE2, J6

Commit message: [enhancement] Rework Power plan.
Parts:
- removed J1003: READER_VDD, Connector_PinHeader_2.54mm:PinHeader_2x03_P2.54mm_Vertical, symbol Connector_Generic:Conn_02x03_Odd_Even
- removed P1001, P523: CMD, Connector_PinHeader_2.54mm:PinHeader_2x02_P2.54mm_Vertical, symbol Connector_Generic:Conn_02x02_Odd_Even
- added D1002, D1003: STPS1L30A, Diode_SMD:D_SMA, symbol Device:D_Schottky_Small_ALT
Connections:
- wire segments 157 -> 150
- no-connect marks 6 -> 4
Other:
- note added: "User can use both external \npower supply and USB power supply."
- moved on the sheet: C1003, C1004, C1005, C4004, D1001, FID1001, FID1002, FID1003, FID1004, FID1005, FID1006, HOLE1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

Commit message: [Fix] General cleanup before production
Connections:
- wire segments 150 -> 152
Changed lines of the file:
@@
 Text Label 15200 7200 2    50   ~ 0
 CW_GND
-Wire Wire Line
-	14750 7200 15200 7200
 Connection ~ 7250 10100
 Text Label 6700 4100 2    50   ~ 0
@@
 Wire Wire Line
 	14000 3800 14100 3800
-Wire Wire Line
-	14100 3500 14750 3500
 Wire Wire Line
 	11900 4950 11900 3600
@@
 	14100 4650 14100 3800
 Connection ~ 14100 3800
-Wire Wire Line
-	14100 3800 14750 3800
 Text Label 14200 3500 0    50   ~ 0
 VDD_CMD
@@
 Text Label 14900 5400 0    50   ~ 0
 VDD_CMD
-Wire Wire Line
-	14750 5400 14900 5400
 Text Label 14750 8150 0    50   ~ 0
 GND_CMD
@@
 Wire Wire Line
 	12700 4050 15400 4050
+Wire Wire Line
+	14100 3500 15600 3500
+Wire Wire Line
+	14750 5400 15600 5400
+Wire Wire Line
+	15600 3500 15600 5400
+Wire Wire Line
+	15700 7200 15700 3800
+Wire Wire Line
+	14100 3800 15700 3800
+Wire Wire Line
+	14750 7200 15700 7200
 $EndSCHEMATC

Commit message: [fix] ground plans => ready for review
Connections:
- net TX_CONSOLE is gone; now on net RX_CONSOLE: U520.6 (VOB)
- net RX_CONSOLE: now also D1001.2 (A), R1002.2
- net CW_GND renamed GND_CMD
